Commit message: BackUp

File: xacro/mini_mec.xacro (robot description, xacro)
@@ -63,10 +63,10 @@
     </xacro:macro>
     <xacro:macro name="shaft_roll_joint" params="LR FR ROLL SHAFT *origin1 *origin2 *axis">
-    <joint name="${LR}_${FR}_${SHAFT}_joint" type="fixed"><!-- type="continuous"-->
+    <joint name="${LR}_${FR}_${SHAFT}_joint" type="continuous"><!-- type="continuous"-->
         <xacro:insert_block name="origin1"/>
         <parent link="${LR}_${FR}_wheel_link"/>
         <child link="${LR}_${FR}_${SHAFT}_link"/>
     </joint>
-    <joint name="${LR}_${FR}_${ROLL}_joint" type="fixed"><!-- type="continuous"-->
+    <joint name="${LR}_${FR}_${ROLL}_joint" type="continuous"><!-- type="continuous"-->
         <xacro:insert_block name="origin2"/>
         <parent link="${LR}_${FR}_${SHAFT}_link"/>
@@ -81,44 +81,44 @@
     </joint>
     <xacro:imu prefix="imu"/>
-    <roll_gazebo LR="left" FR="front" ROLL="roll1"/>
-    <roll_gazebo LR="left" FR="front" ROLL="roll2"/>
-    <roll_gazebo LR="left" FR="front" ROLL="roll3"/>
-    <roll_gazebo LR="left" FR="front" ROLL="roll4"/>
-    <roll_gazebo LR="left" FR="front" ROLL="roll5"/>
-    <roll_gazebo LR="left" FR="front" ROLL="roll6"/>
-    <roll_gazebo LR="left" FR="front" ROLL="roll7"/>
-    <roll_gazebo LR="left" FR="front" ROLL="roll8"/>
-    <roll_gazebo LR="left" FR="front" ROLL="roll9"/>
-    <roll_gazebo LR="left" FR="front" ROLL="roll10"/>
-    <roll_gazebo LR="right" FR="front" ROLL="roll1"/>
-    <roll_gazebo LR="right" FR="front" ROLL="roll2"/>
-    <roll_gazebo LR="right" FR="front" ROLL="roll3"/>
-    <roll_gazebo LR="right" FR="front" ROLL="roll4"/>
-    <roll_gazebo LR="right" FR="front" ROLL="roll5"/>
-    <roll_gazebo LR="right" FR="front" ROLL="roll6"/>
-    <roll_gazebo LR="right" FR="front" ROLL="roll7"/>
-    <roll_gazebo LR="right" FR="front" ROLL="roll8"/>
-    <roll_gazebo LR="right" FR="front" ROLL="roll9"/>
-    <roll_gazebo LR="right" FR="front" ROLL="roll10"/>
-    <roll_gazebo LR="left" FR="rear" ROLL="roll1"/>
-    <roll_gazebo LR="left" FR="rear" ROLL="roll2"/>
-    <roll_gazebo LR="left" FR="rear" ROLL="roll3"/>
-    <roll_gazebo LR="left" FR="rear" ROLL="roll4"/>
-    <roll_gazebo LR="left" FR="rear" ROLL="roll5"/>
-    <roll_gazebo LR="left" FR="rear" ROLL="roll6"/>
-    <roll_gazebo LR="left" FR="rear" ROLL="roll7"/>
-    <roll_gazebo LR="left" FR="rear" ROLL="roll8"/>
-    <roll_gazebo LR="left" FR="rear" ROLL="roll9"/>
-    <roll_gazebo LR="left" FR="rear" ROLL="roll10"/>
-    <roll_gazebo LR="right" FR="rear" ROLL="roll1"/>
-    <roll_gazebo LR="right" FR="rear" ROLL="roll2"/>
-    <roll_gazebo LR="right" FR="rear" ROLL="roll3"/>
-    <roll_gazebo LR="right" FR="rear" ROLL="roll4"/>
-    <roll_gazebo LR="right" FR="rear" ROLL="roll5"/>
-    <roll_gazebo LR="right" FR="rear" ROLL="roll6"/>
-    <roll_gazebo LR="right" FR="rear" ROLL="roll7"/>
-    <roll_gazebo LR="right" FR="rear" ROLL="roll8"/>
-    <roll_gazebo LR="right" FR="rear" ROLL="roll9"/>
-    <roll_gazebo LR="right" FR="rear" ROLL="roll10"/>
+    <xacro:roll_gazebo LR="left" FR="front" ROLL="roll1"/>
+    <xacro:roll_gazebo LR="left" FR="front" ROLL="roll2"/>
+    <xacro:roll_gazebo LR="left" FR="front" ROLL="roll3"/>
+    <xacro:roll_gazebo LR="left" FR="front" ROLL="roll4"/>
+    <xacro:roll_gazebo LR="left" FR="front" ROLL="roll5"/>
+    <xacro:roll_gazebo LR="left" FR="front" ROLL="roll6"/>
+    <xacro:roll_gazebo LR="left" FR="front" ROLL="roll7"/>
+    <xacro:roll_gazebo LR="left" FR="front" ROLL="roll8"/>
+    <xacro:roll_gazebo LR="left" FR="front" ROLL="roll9"/>
+    <xacro:roll_gazebo LR="left" FR="front" ROLL="roll10"/>
+    <xacro:roll_gazebo LR="right" FR="front" ROLL="roll1"/>
+    <xacro:roll_gazebo LR="right" FR="front" ROLL="roll2"/>
+    <xacro:roll_gazebo LR="right" FR="front" ROLL="roll3"/>
+    <xacro:roll_gazebo LR="right" FR="front" ROLL="roll4"/>
+    <xacro:roll_gazebo LR="right" FR="front" ROLL="roll5"/>
+    <xacro:roll_gazebo LR="right" FR="front" ROLL="roll6"/>
+    <xacro:roll_gazebo LR="right" FR="front" ROLL="roll7"/>
+    <xacro:roll_gazebo LR="right" FR="front" ROLL="roll8"/>
+    <xacro:roll_gazebo LR="right" FR="front" ROLL="roll9"/>
+    <xacro:roll_gazebo LR="right" FR="front" ROLL="roll10"/>
+    <xacro:roll_gazebo LR="left" FR="rear" ROLL="roll1"/>
+    <xacro:roll_gazebo LR="left" FR="rear" ROLL="roll2"/>
+    <xacro:roll_gazebo LR="left" FR="rear" ROLL="roll3"/>
+    <xacro:roll_gazebo LR="left" FR="rear" ROLL="roll4"/>
+    <xacro:roll_gazebo LR="left" FR="rear" ROLL="roll5"/>
+    <xacro:roll_gazebo LR="left" FR="rear" ROLL="roll6"/>
+    <xacro:roll_gazebo LR="left" FR="rear" ROLL="roll7"/>
+    <xacro:roll_gazebo LR="left" FR="rear" ROLL="roll8"/>
+    <xacro:roll_gazebo LR="left" FR="rear" ROLL="roll9"/>
+    <xacro:roll_gazebo LR="left" FR="rear" ROLL="roll10"/>
+    <xacro:roll_gazebo LR="right" FR="rear" ROLL="roll1"/>
+    <xacro:roll_gazebo LR="right" FR="rear" ROLL="roll2"/>
+    <xacro:roll_gazebo LR="right" FR="rear" ROLL="roll3"/>
+    <xacro:roll_gazebo LR="right" FR="rear" ROLL="roll4"/>
+    <xacro:roll_gazebo LR="right" FR="rear" ROLL="roll5"/>
+    <xacro:roll_gazebo LR="right" FR="rear" ROLL="roll6"/>
+    <xacro:roll_gazebo LR="right" FR="rear" ROLL="roll7"/>
+    <xacro:roll_gazebo LR="right" FR="rear" ROLL="roll8"/>
+    <xacro:roll_gazebo LR="right" FR="rear" ROLL="roll9"/>
+    <xacro:roll_gazebo LR="right" FR="rear" ROLL="roll10"/>
     <xacro:astra_camera prefix="camera"/>
     <xacro:wheel_joint LR="right" FR="front" >
@@ -174,8 +174,8 @@
           izz="4.60060413465442E-06" />
     </xacro:wheel_link>
-    <transmission_choose LR="right" FR="front" />
-    <transmission_choose LR="left"  FR="front" />
-    <transmission_choose LR="right" FR="rear"  />
-    <transmission_choose LR="left"  FR="rear"  />
+    <xacro:transmission_choose LR="right" FR="front" />
+    <xacro:transmission_choose LR="left"  FR="front" />
+    <xacro:transmission_choose LR="right" FR="rear"  />
+    <xacro:transmission_choose LR="left"  FR="rear"  />
     <xacro:rplidar LA="laser"/>
     <xacro:shaft_link LR="left"  FR="front" SHAFT="shaft1">

Commit message: modified the models in gazebo and rviz

File: xacro/mini_mec.xacro (robot description, xacro)
@@ -54,5 +54,5 @@
     </joint>
     <xacro:macro name="wheel_joint" params="LR FR *origin ">
-    <joint name="${LR}_${FR}_wheel_joint" type="fixed">
+    <joint name="${LR}_${FR}_wheel_joint" type="continuous"><!-- type="continuous"-->
         <xacro:insert_block name="origin"/>
         <parent link="base_link"/>
@@ -63,5 +63,5 @@
     </xacro:macro>
     <xacro:macro name="shaft_roll_joint" params="LR FR ROLL SHAFT *origin1 *origin2 *axis">
-    <joint name="${LR}_${FR}_${SHAFT}_joint" type="continuous"><!-- type="continuous"-->
+    <joint name="${LR}_${FR}_${SHAFT}_joint" type="fixed">
         <xacro:insert_block name="origin1"/>
         <parent link="${LR}_${FR}_wheel_link"/>

File: xacro/minimec_transmission.xacro (robot description, xacro)
@@ -25,8 +25,8 @@
         <type>transmission_interface/SimpleTransmission</type>
         <joint name="${LR}_${FR}_wheel_joint">
-            <hardwareInterface>VelocityJointInterface</hardwareInterface>
+            <hardwareInterface>hardware_interface/VelocityJointInterface</hardwareInterface>
         </joint>
         <actuator name="${LR}_${FR}_wheel_joint_motor">
-            <hardwareInterface>VelocityJointInterface</hardwareInterface>
+            <hardwareInterface>hardware_interface/VelocityJointInterface</hardwareInterface>
             <mechanicalReduction>1</mechanicalReduction>
             <motorTorqueConstant>1</motorTorqueConstant>

Commit message: gazebo simulation

File: xacro/mini_mec.xacro (robot description, xacro)
@@ -1,4 +1,7 @@
 <?xml version="1.0"?>
 <robot name="fritzrobot" xmlns:xacro="http://www.ros.org/wiki/xacro">
+    <!--gpu-->
+    <xacro:arg name="gpu" default="false"/>
+    <xacro:property name="gpu" value="$(arg gpu)" />
     <!--M_PI-->
     <xacro:property name="M_PI" value="3.1415926535897931" />
@@ -11,4 +14,14 @@
     <xacro:property name="rplidar_min_angle" value="-180" />
     <xacro:property name="rplidar_max_angle" value="180" />
+    <!--velodyne description-->
+    <!--velodyne position-->
+    <xacro:property name="velodyne_offset_x" value="0.038632" />
+    <xacro:property name="velodyne_offset_y" value="0.00018237" />
+    <xacro:property name="velodyne_offset_z" value="0.052" />
+    <!--robosense description-->
+    <!--robosense position-->
+    <xacro:property name="robosense_offset_x" value="-0.07" />
+    <xacro:property name="robosense_offset_y" value="0.00018237" />
+    <xacro:property name="robosense_offset_z" value="0.082" />
     <!--camera description-->
     <!--camera position-->
@@ -35,16 +48,18 @@
     <xacro:property name="box_width" value="0.12" />
     <xacro:property name="box_mass"   value="0.082" />
-    <!--robot with rplidar and camera -->
+    <!--robot with rplidar and camera and velodyne-->
     <xacro:include filename="$(find fritzrobot_description)/xacro/minimec_body.xacro" />
-    <xacro:include filename="$(find fritzrobot_description)/xacro/minimec_rplidar.xacro" />
+    <!--xacro:include filename="$(find fritzrobot_description)/xacro/minimec_rplidar.xacro" /-->
     <xacro:include filename="$(find fritzrobot_description)/xacro/minimec_camera.xacro" />
     <xacro:include filename="$(find fritzrobot_description)/xacro/imu.xacro" />
     <xacro:include filename="$(find fritzrobot_description)/xacro/material.xacro" />
     <xacro:include filename="$(find fritzrobot_description)/xacro/minimec_transmission.xacro" />
-    <joint name="rplidar_joint" type="fixed">
+    <xacro:include filename="$(find velodyne_description)/urdf/VLP-16.urdf.xacro"/>
+    <xacro:include filename="$(find robosense_description)/urdf/RS-16.urdf.xacro"/>
+    <!--joint name="rplidar_joint" type="fixed">
         <origin xyz="${rplidar_offset_x} ${rplidar_offset_y} ${rplidar_offset_z}" rpy="0 0 0" />
 	<parent link="base_link"/>
 	<child link="laser_link"/>
-    </joint>
+    </joint-->
     <!-- Attach the camera -->
     <joint name="camera_frame_joint" type="fixed">
@@ -178,5 +193,38 @@
     <xacro:transmission_choose LR="right" FR="rear"  />
     <xacro:transmission_choose LR="left"  FR="rear"  />
-    <xacro:rplidar LA="laser"/>
+    <gazebo>
+        <plugin name="mecanum_move" filename="libgazebo_ros_mecanum_drive.so">
+            <ros>
+                <namespace>fritzrobot</namespace>
+            </ros>
+            <commandTopic>cmd_vel</commandTopic>
+            <odometryTopic>odom</odometryTopic>
+            <odometryFrame>odom</odometryFrame>
+            <publish_odom>false</publish_odom>
+            <publish_odom_tf>false</publish_odom_tf>
+            <LeftFront>left_front_wheel_joint</LeftFront>
+            <RightFront>right_front_wheel_joint</RightFront>
+            <LeftRear>left_rear_wheel_joint</LeftRear>
+            <RightRear>right_rear_wheel_joint</RightRear>
+            <odometryRate>20</odometryRate>
+            <robotBaseFrame>base_footprint</robotBaseFrame>
+            <publishWheelTF>false</publishWheelTF>
+            <publishWheelJointState>false</publishWheelJointState>
+            <WheelTorque>1</WheelTorque>
+            <WheelSeparationW>0.17</WheelSeparationW>
+            <WheelSeparationL>0.24</WheelSeparationL>
+            <wheelAccel>100</wheelAccel>
+            <wheelDiameter>0.075</wheelDiameter>
+            <isRollerModel>true</isRollerModel>
+        </plugin>
+    </gazebo>
+    <!--xacro:rplidar LA="laser"/-->
+    <!-- The collision_range should be bigger than the radius of the Lidar-->
+    <xacro:VLP-16 parent="base_link" name="velodyne" topic="/velodyne_points" hz="10" samples="440" collision_range="0.06" gpu="${gpu}">
+    <origin xyz="${velodyne_offset_x} ${velodyne_offset_y} ${velodyne_offset_z}" rpy="0 0 0" />
+    </xacro:VLP-16>
+    <xacro:RS-16 parent="base_link" name="robosense" topic="/rs_points" hz="20" samples="900" collision_range="0.06"  gpu="${gpu}">
+        <origin xyz="${robosense_offset_x} ${robosense_offset_y} ${robosense_offset_z}" rpy="0 0 0" />
+    </xacro:RS-16>
     <xacro:shaft_link LR="left"  FR="front" SHAFT="shaft1">
         <origin xyz="5.2047E-05 5.6757E-05 -1.8943E-05" rpy="0 0 0"  />

File: xacro/minimec_transmission.xacro (robot description, xacro)
@@ -35,9 +35,9 @@
     </xacro:macro>
   <gazebo>
-    <plugin name="gazebo_ros_control" filename="libgazebo_ros_control.so">
+    <!--plugin name="gazebo_ros_control" filename="libgazebo_ros_control.so">
       <robotNamespace>/fritzrobot</robotNamespace>
       <robotSimType>gazebo_ros_control/DefaultRobotHWSim</robotSimType>
       <legacyModeNS>true</legacyModeNS>
-    </plugin>
+    </plugin-->
   </gazebo>
 </robot>

Commit message: added RS-M1P Lidar

File: xacro/mini_mec.xacro (robot description, xacro)
@@ -23,5 +23,8 @@
     <xacro:property name="robosense_offset_x" value="-0.07" />
     <xacro:property name="robosense_offset_y" value="0.00018237" />
-    <xacro:property name="robosense_offset_z" value="0.082" />
+    <xacro:property name="robosense_offset_z" value="0.083" />
+    <xacro:property name="rs_m1p_offset_x" value="0.038632" />
+    <xacro:property name="rs_m1p_offset_y" value="0.00018237" />
+    <xacro:property name="rs_m1p_offset_z" value="0.083" />
     <!--camera description-->
     <!--camera position-->
@@ -57,4 +60,5 @@
     <xacro:include filename="$(find velodyne_description)/urdf/VLP-16.urdf.xacro"/>
     <xacro:include filename="$(find robosense_description)/urdf/RS-16.urdf.xacro"/>
+    <xacro:include filename="$(find robosense_plugin)/models/RS-M1P.urdf.xacro"/>
     <!--joint name="rplidar_joint" type="fixed">
         <origin xyz="${rplidar_offset_x} ${rplidar_offset_y} ${rplidar_offset_z}" rpy="0 0 0" />
@@ -63,9 +67,9 @@
     </joint-->
     <!-- Attach the camera -->
-    <joint name="camera_frame_joint" type="fixed">
+    <!--joint name="camera_frame_joint" type="fixed">
 	<origin xyz="${camera_offset_x} ${camera_offset_y} ${camera_offset_z}" rpy="0 0 0" />
 	<parent link="base_link"/>
 	<child link="camera_link"/>
-    </joint>
+    </joint-->
     <xacro:macro name="wheel_joint" params="LR FR *origin ">
     <joint name="${LR}_${FR}_wheel_joint" type="continuous"><!-- type="continuous"-->
@@ -136,5 +140,5 @@
     <xacro:roll_gazebo LR="right" FR="rear" ROLL="roll9"/>
     <xacro:roll_gazebo LR="right" FR="rear" ROLL="roll10"/>
-    <xacro:astra_camera prefix="camera"/>
+    <!--xacro:astra_camera prefix="camera"/-->
     <xacro:wheel_joint LR="right" FR="front" >
         <origin xyz="${front_wheel_position_x} ${right_front_wheel_position_y} ${wheel_position_z} " rpy="0 0 0"/>
@@ -221,10 +225,13 @@
     <!--xacro:rplidar LA="laser"/-->
     <!-- The collision_range should be bigger than the radius of the Lidar-->
-    <xacro:VLP-16 parent="base_link" name="velodyne" topic="/velodyne_points" hz="10" samples="440" collision_range="0.06" gpu="${gpu}">
+    <!--xacro:VLP-16 parent="base_link" name="velodyne" topic="/velodyne_points" hz="10" samples="440" collision_range="0.06" gpu="${gpu}">
     <origin xyz="${velodyne_offset_x} ${velodyne_offset_y} ${velodyne_offset_z}" rpy="0 0 0" />
-    </xacro:VLP-16>
-    <xacro:RS-16 parent="base_link" name="robosense" topic="/rs_points" hz="20" samples="900" collision_range="0.06"  gpu="${gpu}">
+    </xacro:VLP-16-->
+    <!--xacro:RS-16 parent="base_link" name="robosense" topic="/rs_points" hz="20" samples="900" collision_range="0.06"  gpu="${gpu}">
         <origin xyz="${robosense_offset_x} ${robosense_offset_y} ${robosense_offset_z}" rpy="0 0 0" />
-    </xacro:RS-16>
+    </xacro:RS-16-->
+    <xacro:RS-M1P parent="base_link" name="RS-M1P" visualize="true">
+        <origin xyz="${rs_m1p_offset_x} ${rs_m1p_offset_y} ${rs_m1p_offset_z}" rpy="0 0 0" />
+    </xacro:RS-M1P>
     <xacro:shaft_link LR="left"  FR="front" SHAFT="shaft1">
         <origin xyz="5.2047E-05 5.6757E-05 -1.8943E-05" rpy="0 0 0"  />
